File: pcb/releases/v0.1.0/anolis-brain-interface.kicad_pcb (KiCad board)
At the start: 2 copper layers, 14 x 18 mm, 27 parts, among them J1 214721-0020, SW1 EVQ-P7A01P, U1 RHD2216, U2 Setebos-I, U3 TPS70933, U4 LTC4054ES5-4.2

Commit message: Fixed inconsistent routing.
Routing:
- net (no net): track 9.77 -> 0.00 mm
- net Net-(U3-IN): track 0.00 -> 9.10 mm
Changed lines of the file:
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@@
     (grid_origin 126 106)
     (pcbplotparams
-      (layerselection 0x00010fc_ffffffff)
+      (layerselection 0x00010cc_ffffffff)
       (plot_on_all_layers_selection 0x0000000_00000000)
       (disableapertmacros false)
-      (usegerberextensions false)
+      (usegerberextensions true)
       (usegerberattributes true)
       (usegerberadvancedattributes true)
@@
       (outputformat 1)
       (mirror false)
-      (drillshape 1)
+      (drillshape 0)
       (scaleselection 1)
-      (outputdirectory "")
+      (outputdirectory "gerber")
     )
   )
@@
     (descr "Resistor SMD 0402 (1005 Metric), square (rectangular) end terminal, IPC_7351 nominal, (Body size source: IPC-SM-782 page 72, https://www.pcb-3d.com/wordpress/wp-content/uploads/ipc-sm-782a_amendment_1_and_2.pdf), generated with kicad-footprint-generator")
     (tags "resistor")
-    (property "Order Number" "755-SFR01MZPF2672")
+    (property "Order Number" "71-CRCW0402-50K-E3")
     (property "Sheetfile" "anolis-brain-interface.kicad_sch")
     (property "Sheetname" "")
@@
     (style (thickness 0.1) (arrow_length 1.27) (text_position_mode 0) (extension_height 0.58642) (extension_offset 0.5) keep_text_aligned)
   )
-  (segment (start 133 83.2) (end 134.1 84.3) (width 0.1) (layer "B.Cu") (net 0))
-  (segment (start 130.4 82.425) (end 129.0875 82.425) (width 0.1) (layer "B.Cu") (net 0))
-  (segment (start 128.85 81.85) (end 128.7 81.7) (width 0.1) (layer "B.Cu") (net 0))
-  (segment (start 128.85 82.6625) (end 128.85 81.85) (width 0.1) (layer "B.Cu") (net 0))
-  (segment (start 128.7 81.7) (end 127.1 81.7) (width 0.1) (layer "B.Cu") (net 0))
-  (segment (start 126.95 81.85) (end 127.1 81.7) (width 0.1) (layer "B.Cu") (net 0))
-  (segment (start 131.175 83.2) (end 133 83.2) (width 0.1) (layer "B.Cu") (net 0))
-  (segment (start 130.4 82.425) (end 131.175 83.2) (width 0.1) (layer "B.Cu") (net 0))
-  (segment (start 129.0875 82.425) (end 128.85 82.6625) (width 0.1) (layer "B.Cu") (net 0))
-  (segment (start 126.95 82.6625) (end 126.95 81.85) (width 0.1) (layer "B.Cu") (net 0))
   (segment (start 135.3 85) (end 135.3 85.8) (width 0.1) (layer "F.Cu") (net 19))
   (segment (start 135.3 85.8) (end 135.9 86.4) (width 0.1) (layer "F.Cu") (net 19))
@@
   (segment (start 128.95 94.95) (end 127.915 95.985) (width 0.1) (layer "F.Cu") (net 44))
   (segment (start 127.915 95.985) (end 126.7 95.985) (width 0.1) (layer "F.Cu") (net 44))
+  (segment (start 133 83.2) (end 134.1 84.3) (width 0.1) (layer "B.Cu") (net 45))
+  (segment (start 126.95 82.6625) (end 126.95 81.85) (width 0.1) (layer "B.Cu") (net 45))
+  (segment (start 127.1 81.7) (end 129.125 81.7) (width 0.1) (layer "B.Cu") (net 45))
+  (segment (start 129.85 82.425) (end 130.4 82.425) (width 0.1) (layer "B.Cu") (net 45))
+  (segment (start 129.125 81.7) (end 129.85 82.425) (width 0.1) (layer "B.Cu") (net 45))
+  (segment (start 131.175 83.2) (end 133 83.2) (width 0.1) (layer "B.Cu") (net 45))
+  (segment (start 130.4 82.425) (end 131.175 83.2) (width 0.1) (layer "B.Cu") (net 45))
+  (segment (start 126.95 81.85) (end 127.1 81.7) (width 0.1) (layer "B.Cu") (net 45))
 )
