File: pcb/anolis-brain-interface.kicad_sch (KiCad schematic)
At the start: 27 parts, among them J1 214721-0020, SW1 EVQ-P7A01P, U1 RHD2216, U2 Setebos-I, U3 TPS70933, U4 LTC4054ES5-4.2

Commit message: PCB version 0.1.0.
Parts:
- C1, C2, C3: Order Number (none) -> 581-KGM15CR51C106KT; Supplier (none) -> Mouser
- C4: renamed from C7; Order Number (none) -> 581-KGM05AR71C104KH; Supplier (none) -> Mouser
- C5: Order Number (none) -> 581-KGM05ACG1E102JH; Supplier (none) -> Mouser
- C6: Order Number (none) -> 581-KGM05AR71C104KH; Supplier (none) -> Mouser
- D2: Order Number (none) -> 710-150040RS73240; Supplier (none) -> Mouser
- R1: Order Number (none) -> 755-SFR01MZPF2672; Supplier (none) -> Mouser
- R2: Order Number (none) -> 71-CRCW0402-1.0K-E3; Supplier (none) -> Mouser
Connections:
- net VIN: no longer C2.1, D1.3, U3.1 (IN), U3.3 (EN)
- new net: C2.1, D1.3, U3.1 (IN)
- no-connect marks 18 -> 24
Changed lines of the file:
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@@
   (title_block
     (title "Anolis Brain Interface")
+    (date "2023-11-20")
+    (rev "0.1.0")
   )
   (junction (at 63.5 149.86) (diameter 0) (color 0 0 0 0)
@@
   )
   (no_connect (at 72.39 96.52))
+  (no_connect (at 62.23 96.52))
   (no_connect (at 181.61 77.47))
   (no_connect (at 77.47 96.52))
+  (no_connect (at 104.14 74.93))
   (no_connect (at 191.77 77.47))
   (no_connect (at 184.15 77.47))
   (no_connect (at 67.31 96.52))
   (no_connect (at 165.1 44.45))
+  (no_connect (at 48.26 85.09))
   (no_connect (at 210.82 59.69))
   (no_connect (at 189.23 77.47))
@@
   (no_connect (at 194.31 77.47))
   (no_connect (at 82.55 96.52))
+  (no_connect (at 90.17 96.52))
   (no_connect (at 165.1 57.15))
   (no_connect (at 186.69 77.47))
   (no_connect (at 210.82 54.61))
   (no_connect (at 210.82 57.15))
+  (no_connect (at 59.69 96.52))
   (no_connect (at 93.98 160.02))
+  (no_connect (at 81.28 160.02))
   (no_connect (at 210.82 52.07))
   (wire (pts (xy 62.23 35.56) (xy 62.23 40.64))
@@
     (stroke (width 0) (type default))
   )
-  (wire (pts (xy 81.28 160.02) (xy 76.2 160.02))
-    (stroke (width 0) (type default))
-  )
   (wire (pts (xy 71.12 154.94) (xy 76.2 154.94))
     (stroke (width 0) (type default))
@@
   )
   (wire (pts (xy 124.46 148.59) (xy 128.27 148.59))
-    (stroke (width 0) (type default))
-  )
-  (wire (pts (xy 76.2 154.94) (xy 76.2 160.02))
     (stroke (width 0) (type default))
   )
@@
       (effects (font (size 1.27 1.27)) hide)
     )
-    (property "Order Number" "" (at 71.12 160.02 0)
-      (effects (font (size 1.27 1.27)) hide)
-    )
-    (property "Supplier" "" (at 71.12 160.02 0)
+    (property "Order Number" "581-KGM15CR51C106KT" (at 71.12 160.02 0)
+      (effects (font (size 1.27 1.27)) hide)
+    )
+    (property "Supplier" "Mouser" (at 71.12 160.02 0)
       (effects (font (size 1.27 1.27)) hide)
     )
@@
       (effects (font (size 1.27 1.27)) hide)
     )
-    (property "Order Number" "" (at 229.87 77.47 0)
-      (effects (font (size 1.27 1.27)) hide)
-    )
-    (property "Supplier" "" (at 229.87 77.47 0)
+    (property "Order Number" "71-CRCW0402-1.0K-E3" (at 229.87 77.47 0)
+      (effects (font (size 1.27 1.27)) hide)
+    )
+    (property "Supplier" "Mouser" (at 229.87 77.47 0)
       (effects (font (size 1.27 1.27)) hide)
     )
@@
       (effects (font (size 1.27 1.27)) hide)
     )
-    (property "Order Number" "" (at 124.46 156.21 0)
-      (effects (font (size 1.27 1.27)) hide)
-    )
-    (property "Supplier" "" (at 124.46 156.21 0)
+    (property "Order Number" "755-SFR01MZPF2672" (at 124.46 156.21 0)
+      (effects (font (size 1.27 1.27)) hide)
+    )
+    (property "Supplier" "Mouser" (at 124.46 156.21 0)
       (effects (font (size 1.27 1.27)) hide)
     )
@@
       (effects (font (size 1.27 1.27)) hide)
     )
-    (property "Order Number" "" (at 229.87 68.58 0)
-      (effects (font (size 1.27 1.27)) hide)
-    )
-    (property "Supplier" "" (at 229.87 68.58 0)
+    (property "Order Number" "710-150040RS73240" (at 229.87 68.58 0)
+      (effects (font (size 1.27 1.27)) hide)
+    )
+    (property "Supplier" "Mouser" (at 229.87 68.58 0)
       (effects (font (size 1.27 1.27)) hide)
     )
@@
       (effects (font (size 1.27 1.27)) hide)
     )
-    (property "Order Number" "" (at 113.03 160.02 0)
-      (effects (font (size 1.27 1.27)) hide)
-    )
-    (property "Supplier" "" (at 113.03 160.02 0)
+    (property "Order Number" "581-KGM15CR51C106KT" (at 113.03 160.02 0)
+      (effects (font (size 1.27 1.27)) hide)
+    )
+    (property "Supplier" "Mouser" (at 113.03 160.02 0)
       (effects (font (size 1.27 1.27)) hide)
     )
@@
       (effects (font (size 1.27 1.27)) hide)
     )
-    (property "Order Number" "" (at 63.5 160.02 0)
-      (effects (font (size 1.27 1.27)) hide)
-    )
-    (property "Supplier" "" (at 63.5 160.02 0)
+    (property "Order Number" "581-KGM15CR51C106KT" (at 63.5 160.02 0)
+      (effects (font (size 1.27 1.27)) hide)
+    )
+    (property "Supplier" "Mouser" (at 63.5 160.02 0)
       (effects (font (size 1.27 1.27)) hide)
     )
@@
       (effects (font (size 1.27 1.27)) hide)
     )
-    (property "Order Number" "" (at 92.71 101.6 0)
-      (effects (font (size 1.27 1.27)) hide)
-    )
-    (property "Supplier" "" (at 92.71 101.6 0)
+    (property "Order Number" "581-KGM05ACG1E102JH" (at 92.71 101.6 0)
+      (effects (font (size 1.27 1.27)) hide)
+    )
+    (property "Supplier" "Mouser" (at 92.71 101.6 0)
       (effects (font (size 1.27 1.27)) hide)
     )
@@
   (symbol (lib_id "Device:C") (at 44.45 88.9 0) (unit 1)
     (in_bom yes) (on_board yes) (dnp no)
-    (property "Reference" "C7" (at 38.1 87.63 0)
+    (property "Reference" "C4" (at 38.1 87.63 0)
       (effects (font (size 1.27 1.27)) (justify left))
     )
@@
       (effects (font (size 1.27 1.27)) hide)
     )
-    (property "Order Number" "" (at 44.45 88.9 0)
-      (effects (font (size 1.27 1.27)) hide)
-    )
-    (property "Supplier" "" (at 44.45 88.9 0)
+    (property "Order Number" "581-KGM05AR71C104KH" (at 44.45 88.9 0)
+      (effects (font (size 1.27 1.27)) hide)
+    )
+    (property "Supplier" "Mouser" (at 44.45 88.9 0)
       (effects (font (size 1.27 1.27)) hide)
     )
@@
       (project "anolis-brain-interface"
         (path "/2073a088-93fe-4857-bf83-cba62e9d9994"
-          (reference "C7") (unit 1)
+          (reference "C4") (unit 1)
         )
       )
@@
       (effects (font (size 1.27 1.27)) hide)
     )
-    (property "Order Number" "" (at 114.3 85.09 0)
-      (effects (font (size 1.27 1.27)) hide)
-    )
-    (property "Supplier" "" (at 114.3 85.09 0)
-      (effects (font (size 1.27 1.27)) hide)
-    )
+    (property "Order Number" "581-KGM05AR71C104KH" (at 114.3 85.09 0)
+      (effects (font (size 1.27 1.27)) hide)
+    )
+    (property "Supplier" "Mouser" (at 114.3 85.09 0)
+      (effects (font (size 1.27 1.27)) hide)
+    )

Commit message: Order number corrected.
Parts:
- R1: Order Number 755-SFR01MZPF2672 -> 71-CRCW0402-50K-E3
Changed lines of the file:
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@@
       (effects (font (size 1.27 1.27)) hide)
     )
-    (property "Order Number" "755-SFR01MZPF2672" (at 124.46 156.21 0)
+    (property "Order Number" "71-CRCW0402-50K-E3" (at 124.46 156.21 0)
       (effects (font (size 1.27 1.27)) hide)
     )

Commit message: Replaced incorrect order number.
Parts:
- C5: Order Number 581-KGM05ACG1E102JH -> 581-04025C103JAT2A
Changed lines of the file:
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@@
       (effects (font (size 1.27 1.27)) hide)
     )
-    (property "Order Number" "581-KGM05ACG1E102JH" (at 92.71 101.6 0)
+    (property "Order Number" "581-04025C103JAT2A" (at 92.71 101.6 0)
       (effects (font (size 1.27 1.27)) hide)
     )
